File: KiCad/SailCam_MK5/SailCam_MK5.sch (KiCad schematic (older format))
At the start: 6 parts, among them J1 B2B-PH-K-SLFSN, J2 B2B-PH-K-SLFSN, J3 B2B-PH-K-SLFSN, J4 B4B-PH-K-SLFSN, J5 SSW-108-02-G-S, J6 SSW-104-02-G-S

Commit message: update
Parts:
- J1, J2, J3: symbol B2B-PH-K-SLFSN:B2B-PH-K-SLFSN -> SailCam_MK5-rescue:B2B-PH-K-SLFSN-B2B-PH-K-SLFSN
- J4: symbol B4B-PH-K-SLFSN:B4B-PH-K-SLFSN -> SailCam_MK5-rescue:B4B-PH-K-SLFSN-B4B-PH-K-SLFSN
- J5: symbol SSW-108-02-G-S:SSW-108-02-G-S -> SailCam_MK5-rescue:SSW-108-02-G-S-SSW-108-02-G-S
- J6: symbol SSW-104-02-G-S:SSW-104-02-G-S -> SailCam_MK5-rescue:SSW-104-02-G-S-SSW-104-02-G-S
Connections:
- net Cam_CS: now also J5.1; no longer J5.8
- net GND: now also J5.5; no longer J5.4
- net MISO: now also J5.3; no longer J5.6
- net MOSI: now also J5.2; no longer J5.7
- net SCK: now also J5.4; no longer J5.5
- net SCL: now also J5.8; no longer J5.1
- net SDA: now also J5.7; no longer J5.2
- net VCC: now also J5.6; no longer J5.3
Changed lines of the file:
@@
 $EndDescr
 $Comp
-L SSW-108-02-G-S:SSW-108-02-G-S J5
+L SailCam_MK5-rescue:SSW-108-02-G-S-SSW-108-02-G-S J5
 U 1 1 61092C68
 P 1950 3600
@@
 	1    0    0    -1
 $EndComp
+Text Label 1950 3600 2    50   ~ 0
+Cam_CS
+Text Label 1950 3700 2    50   ~ 0
+MOSI
+Text Label 1950 3800 2    50   ~ 0
+MISO
+Text Label 1950 3900 2    50   ~ 0
+SCK
+Text Label 1950 4000 2    50   ~ 0
+GND
+Text Label 1950 4100 2    50   ~ 0
+Vcc
+Text Label 1950 4200 2    50   ~ 0
+SDA
 Text Label 1950 4300 2    50   ~ 0
-Cam_CS
-Text Label 1950 4200 2    50   ~ 0
-MOSI
-Text Label 1950 4100 2    50   ~ 0
-MISO
-Text Label 1950 4000 2    50   ~ 0
-SCK
-Text Label 1950 3900 2    50   ~ 0
-GND
-Text Label 1950 3800 2    50   ~ 0
-VCC
-Text Label 1950 3700 2    50   ~ 0
-SDA
-Text Label 1950 3600 2    50   ~ 0
 SCL
 $Comp
-L B2B-PH-K-SLFSN:B2B-PH-K-SLFSN J3
+L SailCam_MK5-rescue:B2B-PH-K-SLFSN-B2B-PH-K-SLFSN J3
 U 1 1 61095DC0
 P 1950 2600
@@
 $EndComp
 $Comp
-L SSW-104-02-G-S:SSW-104-02-G-S J6
+L SailCam_MK5-rescue:SSW-104-02-G-S-SSW-104-02-G-S J6
 U 1 1 610EDBD8
 P 1950 4600
@@
 SDA
 $Comp
-L B4B-PH-K-SLFSN:B4B-PH-K-SLFSN J4
+L SailCam_MK5-rescue:B4B-PH-K-SLFSN-B4B-PH-K-SLFSN J4
 U 1 1 6110A6B6
 P 1950 3000
@@
 F3 "GND" I L 8600 2550 50
 F4 "Vcc" I L 8600 2450 50
-F5 "EN" I R 9650 2350 50
-F6 "OUT" I R 9650 2450 50
+F5 "OUT" I R 9650 2450 50
+F6 "OpAmpEN" I R 9650 2550 50
 $EndSheet
 Text Label 8600 2550 2    50   ~ 0
@@
 $EndSheet
 $Sheet
-S 8600 1500 750  400
+S 8600 1350 750  500
 U 611BA1F2
 F0 "PowerSupply" 50
 F1 "SailCam_MK5_PowerSupply.sch" 50
-F2 "Vcc" I L 8600 1600 50
-F3 "GND" I L 8600 1700 50
-F4 "Vcc_5v" I R 9350 1600 50
-F5 "CHG" I R 9350 1800 50
-F6 "Vcc_Bat" I L 8600 1800 50
-F7 "Vcc_5v_S" I R 9350 1700 50
+F2 "Vcc" I L 8600 1450 50
+F3 "GND" I L 8600 1550 50
+F4 "Vcc_5v" I R 9350 1450 50
+F5 "CHG" I R 9350 1650 50
+F6 "Vcc_Bat" I L 8600 1650 50
+F7 "Vcc_5v_S" I R 9350 1550 50
+F8 "Bat_Chg_Vcc" I L 8600 1750 50
 $EndSheet
 $Sheet
@@
 $EndSheet
 $Comp
-L B2B-PH-K-SLFSN:B2B-PH-K-SLFSN J2
+L SailCam_MK5-rescue:B2B-PH-K-SLFSN-B2B-PH-K-SLFSN J2
 U 1 1 611F6EFF
 P 1950 2200
@@
 Text Label 1950 2300 2    50   ~ 0
 Vcc_5v_S
-Text Label 9350 1600 0    50   ~ 0
-Vcc_5v
-Text Label 9350 1700 0    50   ~ 0
+Text Label 9350 1450 0    50   ~ 0
+Vcc_5v
+Text Label 9350 1550 0    50   ~ 0
 Vcc_5v_S
-Text Label 8600 1800 2    50   ~ 0
+Text Label 8600 1650 2    50   ~ 0
 Vcc_Bat
-Text Label 8600 1700 2    50   ~ 0
-GND
-Text Label 8600 1600 2    50   ~ 0
+Text Label 8600 1550 2    50   ~ 0
+GND
+Text Label 8600 1450 2    50   ~ 0
 Vcc
 Text Label 8600 3200 2    50   ~ 0
@@
 Text Label 8600 3850 2    50   ~ 0
 NEMA-
-Text Label 9350 1800 0    50   ~ 0
+Text Label 9350 1650 0    50   ~ 0
 CHG
 Text Label 9650 2450 0    50   ~ 0
@@
 Text Label 10850 6150 2    50   ~ 0
 GND
-$Sheet
-S 5950 1500 750  1100
-U 61217E38
-F0 "Micro" 50
-F1 "SailCam_MK5_Micro.sch" 50
-F2 "Vcc" I L 5950 1600 50
-F3 "GND" I L 5950 1700 50
-F4 "CHG" I L 5950 1800 50
-F5 "Rx" I R 6700 1600 50
-F6 "Tx" I R 6700 1700 50
-F7 "SDA" I R 6700 1850 50
-F8 "SCL" I R 6700 1950 50
-F9 "MISO" I R 6700 2100 50
-F10 "MOSI" I R 6700 2200 50
-F11 "SD_CS" I L 5950 1950 50
-F12 "Cam_CS" I L 5950 2050 50
-F13 "SCK" I R 6700 2300 50
-F14 "ADC0" I L 5950 2200 50
-F15 "OpAmpEN" I L 5950 2300 50
-F16 "IR_CTL" I L 5950 2400 50
-F17 "Vcc_5v" I L 5950 2500 50
-$EndSheet
 Text Label 5950 1600 2    50   ~ 0
 Vcc
 Text Label 5950 1700 2    50   ~ 0
 GND
-Text Label 5950 1800 2    50   ~ 0
-CHG
 Text Label 5950 1950 2    50   ~ 0
 SD_CS
@@
 Text Label 6700 1600 0    50   ~ 0
 NEMA_Tx
-Text Label 9650 2350 0    50   ~ 0
+Text Label 9650 2550 0    50   ~ 0
 OpAmpEN
 Text Label 5950 2200 2    50   ~ 0
@@
 MISO
 $Comp
-L B2B-PH-K-SLFSN:B2B-PH-K-SLFSN J1
+L SailCam_MK5-rescue:B2B-PH-K-SLFSN-B2B-PH-K-SLFSN J1
 U 1 1 6129E01E
 P 1950 1800
@@
 Text Label 5950 2500 2    50   ~ 0
 Vcc_5v
+$Sheet
+S 5950 1500 750  1250
+U 61217E38
+F0 "Micro" 50
+F1 "SailCam_MK5_Micro.sch" 50
+F2 "Vcc" I L 5950 1600 50
+F3 "GND" I L 5950 1700 50
+F4 "Rx" I R 6700 1600 50
+F5 "Tx" I R 6700 1700 50
+F6 "SDA" I R 6700 1850 50
+F7 "SCL" I R 6700 1950 50
+F8 "MISO" I R 6700 2100 50
+F9 "MOSI" I R 6700 2200 50
+F10 "SD_CS" I L 5950 1950 50
+F11 "Cam_CS" I L 5950 2050 50
+F12 "SCK" I R 6700 2300 50
+F13 "ADC0" I L 5950 2200 50
+F14 "OpAmpEN" I L 5950 2300 50
+F15 "IR_CTL" I L 5950 2400 50
+F16 "Vcc_5v" I L 5950 2500 50
+F17 "Bat_Chg_Vcc" I L 5950 2600 50
+$EndSheet
+Text Label 5950 2600 2    50   ~ 0
+Bat_Chg_Vcc
+Text Label 8600 1750 2    50   ~ 0
+Bat_Chg_Vcc
 $EndSCHEMATC
