File: KiCad/SailCam_MK5/SailCam_MK5_NEMAInterface.sch (KiCad schematic (older format))
At the start: 8 parts, among them U6 MAX485CSA+, U7 SM712.TCT

Commit message: update
Parts:
- U6: symbol MAX485CSA&plus_:MAX485CSA+ -> SailCam_MK5-rescue:MAX485CSA+-MAX485CSA&plus_
- U7: symbol SM712-TCT:SM712.TCT -> SailCam_MK5-rescue:SM712.TCT-SM712-TCT
Changed lines of the file:
@@
 	6150 3800 6150 4000
 $Comp
-L SM712-TCT:SM712.TCT U7
+L SailCam_MK5-rescue:SM712.TCT-SM712-TCT U7
 U 1 1 611B5A15
 P 7000 3900
@@
 $EndComp
 $Comp
-L MAX485CSA&plus_:MAX485CSA+ U6
+L SailCam_MK5-rescue:MAX485CSA+-MAX485CSA&plus_ U6
 U 1 1 611B5A2E
 P 4400 3700
