File: KiCad/SailCam_MK5/SailCam_MK5_RealTimeClock.sch (KiCad schematic (older format))
At the start: 6 parts, among them U2 DS1672S-33+T&R, Y1 ABS25-32.768KHZ-6-1-T

Commit message: update
Parts:
- B1: symbol BU2032SM-BT-GTR:BU2032SM-BT-GTR -> SailCam_MK5-rescue:BU2032SM-BT-GTR-BU2032SM-BT-GTR
- U2: symbol ds1672:DS1672S-33+T&R -> SailCam_MK5-rescue:DS1672S-33+T&R-ds1672
- Y1: symbol ABS25-32.768KHZ-6-1-T:ABS25-32.768KHZ-6-1-T -> SailCam_MK5-rescue:ABS25-32.768KHZ-6-1-T-ABS25-32.768KHZ-6-1-T
Changed lines of the file:
@@
 $EndDescr
 $Comp
-L ds1672:DS1672S-33+T&R U?
+L SailCam_MK5-rescue:DS1672S-33+T&R-ds1672 U?
 U 1 1 611A5679
 P 5200 3800
@@
 $EndComp
 $Comp
-L ABS25-32.768KHZ-6-1-T:ABS25-32.768KHZ-6-1-T Y?
+L SailCam_MK5-rescue:ABS25-32.768KHZ-6-1-T-ABS25-32.768KHZ-6-1-T Y?
 U 1 1 611A5681
 P 4900 3800
@@
 $EndComp
 $Comp
-L BU2032SM-BT-GTR:BU2032SM-BT-GTR B?
+L SailCam_MK5-rescue:BU2032SM-BT-GTR-BU2032SM-BT-GTR B?
 U 1 1 611A568F
 P 3950 3800
