File: KiCad/SailCam_MK5/SailCam_MK5.kicad_pcb (KiCad board)
At the start: 4 copper layers, 65 x 65 mm, 70 parts, among them J1 B2B-PH-K-SLFSN, J2 B2B-PH-K-SLFSN, J3 B2B-PH-K-SLFSN, J4 B4B-PH-K-SLFSN, J5 SSW-108-02-G-S, J6 SSW-104-02-G-S, J7 USB_B, J8 DM3BT-DSF-PEJS, M1 2491, Q1 SS8050-G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

Commit message: update
Parts:
- Q3: footprint footprints:NCV7805BD2TG -> custom:TO228P1003X240-3N
- U1: value ADA4806-1ARJZ-R7 -> ADA4841-1YRZ-R7; footprint footprints:ADA4806-1ARJZ-R7 -> custom:ADA4841-1YRZ-R7
- moved R4 6.57 mm to (110.0, 86.4), turned to 0 degrees
- moved R3 5.85 mm to (110.0, 89.7)
- moved R2 2.73 mm to (116.6, 77.6)
- moved R1 2.49 mm to (121.1, 77.6)
- moved R22 1.39 mm to (116.1, 97.8)
- moved U1 1.19 mm to (115.4, 82.7)
- moved Q3 0.83 mm to (130.6, 90.5), turned to 180 degrees
Connections:
- C2 pad 1: Net-(C2-Pad1) -> /Bat_Chg_Vcc
- C7 pad 1: /CHG -> /Bat_Chg_Vcc
- J5 pad 1: /SCL -> /Cam_CS
- J5 pad 2: /SDA -> /MOSI
- J5 pad 3: VCC -> /MISO
- J5 pad 4: GND -> /SCK
- J5 pad 5: /SCK -> GND
- J5 pad 6: /MISO -> VCC
- J5 pad 7: /MOSI -> /SDA
- J5 pad 8: /Cam_CS -> /SCL
- J7 pad 1: /CHG -> /Bat_Chg_Vcc
- M1 pad 10: /Cam_CS -> /OpAmpEN
- M1 pad 12: /Micro/GPIO0 -> /SD_CS
- M1 pad 4: /SD_CS -> /Cam_CS
- Q2 pad 3: /Micro/GPIO0 -> /SD_CS
- R16 pad 2: /Micro/GPIO0 -> /SD_CS
- R22 pad 1: /Cam_CS -> /OpAmpEN
- S3 pad 1: /Micro/GPIO0 -> /SD_CS
- U1 pad 1: /ADC0 -> Net-(U1-Pad1)
- U1 pad 2: Net-(U1-Pad2) -> /ADC0
- U1 pad 3: GND -> Net-(R1-Pad2)
- U1 pad 4: Net-(R1-Pad2) -> GND
- U1 pad 5: /ADC0 -> Net-(U1-Pad5)
- U1 pad 6: VCC -> /ADC0
- U1 pad 7: /OpAmpEN -> VCC
- U1 pad 8: VCC -> /OpAmpEN
- U3 pad 3: Net-(C2-Pad1) -> /Bat_Chg_Vcc
- U4 pad 4: Net-(C2-Pad1) -> /Bat_Chg_Vcc
- U8 pad 16: /CHG -> /Bat_Chg_Vcc
- U9 pad 3: /MicroSD/SD_MISO -> /MicroSD/SD_MOSI
- U9 pad 4: /MicroSD/SD_MOSI -> /MicroSD/SD_MISO
Routing:
- net /Bat_Chg_Vcc: track 0.00 -> 138.6 mm, vias 0 -> 2
- net /SD_CS: track 19.1 -> 105.9 mm, vias 1 -> 2
- net /Micro/GPIO0: track 76.8 -> 0.00 mm, vias 1 -> 0
- net Net-(C2-Pad1): track 44.4 -> 0.00 mm, vias 2 -> 0
- net /OpAmpEN: track 0.00 -> 42.4 mm, vias 0 -> 1
- net /CHG: track 74.2 -> 35.9 mm
- net /Cam_CS: track 36.0 -> 24.6 mm
- net /MOSI: track 34.8 -> 23.4 mm, vias 2 -> 1
- net /SDA: track 85.4 -> 78.0 mm
- net GND: track 151.9 -> 144.6 mm, vias 12 -> 11
- net /ADC0: track 57.9 -> 63.7 mm
- net /SCL: track 86.9 -> 82.3 mm
- net VCC: track 200.9 -> 205.3 mm
- net Net-(Q3-Pad1): track 9.17 -> 13.2 mm
- net /Vcc_5v_S: track 98.2 -> 94.2 mm
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Other:
- board text added: "SailCam MK5.2 Tyler Thompson Octana Laboratories"
- board text removed: "SailCam MK5 Tyler Thompson Octana Laboratories"

Commit message: mk5.2
Parts:
- removed S2, S3: SW_Push, Button_Switch_THT:SW_PUSH_6mm
- added G***: LOGO, custom:octana_laboratories_logo, B.Cu at (147.6, 105.9)
- C10, C8, Q3, R16, R17, R18, R19, R20, R21, R25: moved to F.Cu
- J7: value USB_B -> USB_B_Mini; footprint footprints:AMPHENOL_61729-1011BLF -> digikey-footprints:USB_Mini_B_Female_548190519
- R26: footprint Resistor_THT:R_Axial_DIN0411_L9.9mm_D3.6mm_P12.70mm_Horizontal -> Resistor_THT:R_Axial_DIN0207_L6.3mm_D2.5mm_P10.16mm_Horizontal
- U3: moved to B.Cu
- moved C3 60.5 mm to (162.0, 85.8), turned to 90 degrees
- moved R11 49.2 mm to (102.9, 86.5), turned to 0 degrees
- moved R15 46.8 mm to (102.9, 90.9)
- moved D1 45.7 mm to (157.2, 93.5)
- moved R8 45.2 mm to (152.5, 93.5)
- moved R13 45.1 mm to (102.9, 93.1)
- moved J3 44.0 mm to (149.5, 90.3), turned to 90 degrees
- moved R12 43.8 mm to (108.2, 70.9), turned to 90 degrees
- moved R14 41.4 mm to (110.4, 70.9), turned to 90 degrees
- moved R10 40.9 mm to (102.9, 88.7), turned to 0 degrees
- moved U7 37.3 mm to (109.3, 66.3), turned to 0 degrees
- moved R16 35.5 mm to (111.8, 97.5), turned to 0 degrees
- moved C2 35.0 mm to (137.1, 96.7)
- moved R17 34.6 mm to (111.8, 95.3), turned to 0 degrees
- moved U6 34.3 mm to (109.3, 77.9), turned to 90 degrees
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Connections:
- C1 pad 1: VCC -> /CHG
- C1 pad 2: /CHG -> GND
- J7 pad 4: GND -> Net-(J7-Pad4)
Routing:
- net /Bat_Chg_Vcc: track 138.6 -> 55.3 mm
- net GND: track 144.6 -> 84.5 mm, vias 11 -> 6
- net VCC: track 205.3 -> 156.5 mm, vias 6 -> 4
- net Net-(R8-Pad1): track 2.38 -> 40.2 mm
- net /Vcc_5v_S: track 94.2 -> 57.7 mm, vias 1 -> 0
- net Net-(R9-Pad2): track 2.38 -> 37.5 mm, vias 0 -> 2
- net /Micro/RST: track 106.4 -> 76.3 mm, vias 1 -> 2
- net /Micro/GPIO2: track 21.3 -> 50.2 mm, vias 0 -> 2
- net Net-(R12-Pad2): track 6.80 -> 35.4 mm, vias 0 -> 2
- net Net-(R14-Pad2): track 6.80 -> 34.9 mm, vias 0 -> 2
- net /NEMA+: track 31.2 -> 57.7 mm
- net Net-(M1-Pad3): track 3.52 -> 23.6 mm, vias 0 -> 1
- net /OpAmpEN: track 42.4 -> 62.0 mm, vias 1 -> 2
- net /SD_CS: track 105.9 -> 87.2 mm
- net /Vcc_5v: track 124.6 -> 107.0 mm, vias 3 -> 0
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- removed copper zone on In1.Cu, net GND
Other:
- copper layers 4 -> 2
- board text added: "SailCam MK5.2 Tyler Thompson"
- board text removed: "SailCam MK5.2 Tyler Thompson Octana Laboratories"

Commit message: hardward bug fixes
Parts:
- removed C9: 0.1 uF, footprints:C_0805_2012Metric_Pad1.15x1.40mm_HandSolder_FullSilk
- added R27: 10 KΩ, footprints:C_0805_2012Metric_Pad1.15x1.40mm_HandSolder_FullSilk, F.Cu at (111.8, 104.1)
- moved C7 20.7 mm to (156.4, 104.5), turned to 90 degrees
- moved G*** 1.90 mm to (149.5, 105.9)
- moved C10 0.30 mm to (111.8, 108.5)
- moved C8 0.30 mm to (111.8, 106.3)
Connections:
- C7 pad 1: /Bat_Chg_Vcc -> VCC
- J8 pad 10: Net-(J8-Pad10) -> GND
- U8 pad 16: /Bat_Chg_Vcc -> VCC
- U8 pad 4: Net-(C9-Pad1) -> VCC
- U9 pad 15: GND -> Net-(J8-Pad9)
Routing:
- net Net-(J8-Pad9): track 0.00 -> 37.2 mm, vias 0 -> 2
- net VCC: track 156.5 -> 192.5 mm, vias 4 -> 6
- net /Micro/RST: track 76.3 -> 85.1 mm
- net GND: track 84.5 -> 89.7 mm
- net /Bat_Chg_Vcc: track 55.3 -> 50.5 mm
- net Net-(C9-Pad1): track 4.28 -> 0.00 mm
Other:
- outline, holes or cut-outs redrawn
- board text added: "SailCam MK5.3 PN: 014-0003"
- board text removed: "SailCam MK5.2 Tyler Thompson"
