File: KiCad/SailCam_MK5/SailCam_MK5_Micro.sch (KiCad schematic (older format))
At the start: 27 parts, among them J7 USB_B, M1 2491, Q1 SS8050-G, Q2 SS8050-G, Q3 AOD1N60, U8 CH340G, Y2 ECS-120-20-4X

Commit message: update
Parts:
- Q3: footprint TO228P1003X240-3N -> custom:TO228P1003X240-3N; symbol AOD1N60:AOD1N60 -> SailCam_MK5-rescue:AOD1N60-AOD1N60
- U8: symbol CH340G_Interface_USB:CH340G -> SailCam_MK5-rescue:CH340G-CH340G_Interface_USB
Connections:
- net Cam_CS: now also M1.4 (IO16); no longer M1.10 (IO15), R22.1
- net OpAmpEN: now also M1.10 (IO15), R22.1; no longer M1.12 (IO0), Q2.3 (C), R16.2, S3.1
- net SD_CS: now also M1.12 (IO0), Q2.3 (C), R16.2, S3.1; no longer M1.4 (IO16)
- net CHG renamed Bat_Chg_Vcc
Changed lines of the file:
@@
 $Descr A4 11693 8268
 encoding utf-8
-Sheet 6 7
+Sheet 7 7
 Title "SailCam"
 Date "2021-07-31"
@@
 Text Label 6450 3000 0    50   ~ 0
 SCK
-Text Label 6450 2900 0    50   ~ 0
+Text Label 6450 2800 0    50   ~ 0
 Cam_CS
-Text Label 6450 2800 0    50   ~ 0
+Text Label 5650 2800 2    50   ~ 0
 SD_CS
 Text Label 5650 2500 2    50   ~ 0
@@
 $EndComp
 $Comp
-L CH340G_Interface_USB:CH340G U?
+L SailCam_MK5-rescue:CH340G-CH340G_Interface_USB U?
 U 1 1 6121FD94
 P 6050 4600
@@
 NoConn ~ 6450 4500
 Text Label 5250 4350 0    50   ~ 0
-CHG
+Bat_Chg_Vcc
 Wire Wire Line
 	5250 4350 5450 4350
@@
 	7300 5050 7800 5050
 Connection ~ 7300 4650
-Text Label 5650 2800 2    50   ~ 0
-GPIO0
+Text Label 6450 2900 0    50   ~ 0
+OpAmpEN
 Text Label 7950 5450 0    50   ~ 0
-GPIO0
+SD_CS
 Wire Wire Line
 	7950 5450 7800 5450
@@
 Text HLabel 3300 3200 0    50   Input ~ 0
 GND
-Text HLabel 3300 3300 0    50   Input ~ 0
-CHG
 Text HLabel 3300 3400 0    50   Input ~ 0
 Rx
@@
 Text Label 3300 3200 0    50   ~ 0
 GND
-Text Label 3300 3300 0    50   ~ 0
-CHG
 Text Label 3300 3500 0    50   ~ 0
 Tx0
@@
 RST
 Text Label 9200 2600 2    50   ~ 0
-GPIO0
+SD_CS
 Text HLabel 3300 4300 0    50   Input ~ 0
 ADC0
@@
 GPIO2
 Text Label 3300 4400 0    50   ~ 0
-GPIO0
-$Comp
-L AOD1N60:AOD1N60 Q3
+OpAmpEN
+$Comp
+L SailCam_MK5-rescue:AOD1N60-AOD1N60 Q3
 U 1 1 612A588A
 P 10050 4450
 F 0 "Q3" H 10258 4541 50  0000 L CNN
 F 1 "AOD1N60" H 10258 4450 50  0000 L CNN
-F 2 "TO228P1003X240-3N" H 10050 4450 50  0001 L BNN
+F 2 "custom:TO228P1003X240-3N" H 10050 4450 50  0001 L BNN
 F 3 "" H 10050 4450 50  0001 L BNN
 F 4 "IPC 7351B" H 10050 4450 50  0001 L BNN "STANDARD"
@@
 Wire Wire Line
 	9900 4550 9950 4550
+Text HLabel 3300 4700 0    50   Input ~ 0
+Bat_Chg_Vcc
+Text Label 3300 4700 0    50   ~ 0
+Bat_Chg_Vcc
 $EndSCHEMATC

Commit message: mk5.2
Parts:
- removed J7: USB_B, footprints:AMPHENOL_61729-1011BLF, symbol Connector:USB_B
- removed S2, S3: SW_Push, Button_Switch_THT:SW_PUSH_6mm, symbol Switch:SW_Push
- added J7: USB_B_Mini, digikey-footprints:USB_Mini_B_Female_548190519, symbol SailCam:USB_B_Micro
Connections:
- net Bat_Chg_Vcc: now also J7.1 (VBUS)
- net GND: now also J7.5 (GND), J7.SH (Shield)
- net at U8.5 (UD+): now also J7.3 (D+)
- net at U8.6 (UD-): now also J7.2 (D-)
- no-connect marks 5 -> 6
Changed lines of the file:
@@
-$EndComp
-$Comp
-L Connector:USB_B J?
-U 1 1 6121FD9A
-P 4950 4550
-AR Path="/6121FD9A" Ref="J?"  Part="1"
-AR Path="/61217E38/6121FD9A" Ref="J7"  Part="1"
-F 0 "J7" H 5007 5017 50  0000 C CNN
-F 1 "USB_B" H 5007 4926 50  0000 C CNN
-F 2 "footprints:AMPHENOL_61729-1011BLF" H 5100 4500 50  0001 C CNN
-F 3 "https://www.amphenol-icc.com/media/wysiwyg/files/drawing/61729.pdf" H 5100 4500 50  0001 C CNN
-	1    4950 4550
-	1    0    0    -1
 $EndComp
 $Comp
@@
 	4850 4950 4950 4950
 Connection ~ 4950 4950
-Wire Wire Line
-	5250 4550 5650 4550
-Wire Wire Line
-	5650 4650 5250 4650
 $Comp
 L power:GND #PWR?
@@
 	1    0    0    -1
 $EndComp
-Wire Wire Line
-	4050 5250 5250 5250
 Connection ~ 4050 5250
 Wire Wire Line
@@
 	5350 4850 5650 4850
 Connection ~ 4050 5550
-Wire Wire Line
-	5250 4750 5650 4750
-Wire Wire Line
-	5250 4750 5250 5250
 $Comp
 L Device:Q_NPN_BEC Q1
@@
 Wire Wire Line
 	6450 2400 7050 2400
-$Comp
-L Switch:SW_Push S2
-U 1 1 61289747
-P 8500 2800
-F 0 "S2" V 8409 2948 50  0000 L CNN
-F 1 "SW_Push" V 8500 2948 50  0000 L CNN
-F 2 "Button_Switch_THT:SW_PUSH_6mm" H 8500 3000 50  0001 C CNN
-F 3 "~" H 8500 3000 50  0001 C CNN
-F 4 "Reset" V 8591 2948 50  0000 L CNN "Description"
-	1    8500 2800
-	0    1    1    0
-$EndComp
-$Comp
-L power:GND #PWR?
-U 1 1 6128AA66
-P 8500 3000
-AR Path="/6128AA66" Ref="#PWR?"  Part="1"
-AR Path="/611BA1F2/6128AA66" Ref="#PWR?"  Part="1"
-AR Path="/61217E38/6128AA66" Ref="#PWR015"  Part="1"
-F 0 "#PWR015" H 8500 2750 50  0001 C CNN
-F 1 "GND" H 8505 2827 50  0000 C CNN
-F 2 "" H 8500 3000 50  0001 C CNN
-F 3 "" H 8500 3000 50  0001 C CNN
-	1    8500 3000
-	1    0    0    -1
-$EndComp
-$Comp
-L Switch:SW_Push S3
-U 1 1 6128D069
-P 9200 2800
-F 0 "S3" V 9109 2948 50  0000 L CNN
-F 1 "SW_Push" V 9200 2948 50  0000 L CNN
-F 2 "Button_Switch_THT:SW_PUSH_6mm" H 9200 3000 50  0001 C CNN
-F 3 "~" H 9200 3000 50  0001 C CNN
-F 4 "Flash" V 9291 2948 50  0000 L CNN "Description"
-	1    9200 2800
-	0    1    1    0
-$EndComp
-$Comp
-L power:GND #PWR?
-U 1 1 6128D06F
-P 9200 3000
-AR Path="/6128D06F" Ref="#PWR?"  Part="1"
-AR Path="/611BA1F2/6128D06F" Ref="#PWR?"  Part="1"
-AR Path="/61217E38/6128D06F" Ref="#PWR017"  Part="1"
-F 0 "#PWR017" H 9200 2750 50  0001 C CNN
-F 1 "GND" H 9205 2827 50  0000 C CNN
-F 2 "" H 9200 3000 50  0001 C CNN
-F 3 "" H 9200 3000 50  0001 C CNN
-	1    9200 3000
-	1    0    0    -1
-$EndComp
-Text Label 8500 2600 2    50   ~ 0
-RST
-Text Label 9200 2600 2    50   ~ 0
-SD_CS
 Text HLabel 3300 4300 0    50   Input ~ 0
 ADC0
@@
 Text Label 3300 4700 0    50   ~ 0
 Bat_Chg_Vcc
+$Comp
+L SailCam:USB_B_Micro J7
+U 1 1 614CF04D
+P 4950 4550
+F 0 "J7" H 5007 5017 50  0000 C CNN
+F 1 "USB_B_Mini" H 5007 4926 50  0000 C CNN
+F 2 "digikey-footprints:USB_Mini_B_Female_548190519" H 5100 4500 50  0001 C CNN
+F 3 "~" H 5100 4500 50  0001 C CNN
+	1    4950 4550
+	1    0    0    -1
+$EndComp
+Wire Wire Line
+	5650 4750 5300 4750
+Wire Wire Line
+	5300 4750 5300 5250
+Wire Wire Line
+	4050 5250 5300 5250
+NoConn ~ 5250 4750
+Wire Wire Line
+	5250 4650 5650 4650
+Wire Wire Line
+	5250 4550 5650 4550
 $EndSCHEMATC

Commit message: hardward bug fixes
Parts:
- removed C9: 0.1 uF, footprints:C_0805_2012Metric_Pad1.15x1.40mm_HandSolder_FullSilk, symbol Device:C_Small
Connections:
- net Bat_Chg_Vcc: no longer C7.1, U8.16 (VCC)
- net Vcc: now also C7.1, U8.16 (VCC), U8.4 (V3)
Changed lines of the file:
@@
 Bat_Chg_Vcc
 Wire Wire Line
-	5250 4350 5450 4350
-Wire Wire Line
-	5450 4350 5450 4200
-Wire Wire Line
 	5450 4200 5650 4200
-$Comp
-L Device:C_Small C?
-U 1 1 6122930C
-P 5550 5700
-AR Path="/6122930C" Ref="C?"  Part="1"
-AR Path="/61217E38/6122930C" Ref="C9"  Part="1"
-F 0 "C9" H 5642 5746 50  0000 L CNN
-F 1 "0.1 uF" H 5642 5655 50  0000 L CNN
-F 2 "footprints:C_0805_2012Metric_Pad1.15x1.40mm_HandSolder_FullSilk" H 5550 5700 50  0001 C CNN
-F 3 "~" H 5550 5700 50  0001 C CNN
-	1    5550 5700
-	1    0    0    -1
-$EndComp
-$Comp
-L power:GND #PWR?
-U 1 1 61229E38
-P 5550 5800
-AR Path="/61229E38" Ref="#PWR?"  Part="1"
-AR Path="/611BA1F2/61229E38" Ref="#PWR?"  Part="1"
-AR Path="/61217E38/61229E38" Ref="#PWR011"  Part="1"
-F 0 "#PWR011" H 5550 5550 50  0001 C CNN
-F 1 "GND" H 5555 5627 50  0000 C CNN
-F 2 "" H 5550 5800 50  0001 C CNN
-F 3 "" H 5550 5800 50  0001 C CNN
-	1    5550 5800
-	1    0    0    -1
-$EndComp
-Wire Wire Line
-	5550 4300 5650 4300
 $Comp
 L Device:C_Small C?
@@
 $EndComp
 Wire Wire Line
-	5550 4300 5550 5600
-Wire Wire Line
 	5150 5600 5450 5600
-Wire Wire Line
-	5450 5600 5450 4350
-Connection ~ 5450 4350
 $Comp
 L Device:Crystal Y2
@@
 Wire Wire Line
 	5250 4550 5650 4550
+Wire Wire Line
+	5450 4200 5450 5600
+Text Label 5650 4200 2    50   ~ 0
+Vcc
+Wire Wire Line
+	5650 4300 5650 4200
+Connection ~ 5650 4200
 $EndSCHEMATC
