File: KiCad/SailCam_MK5/SailCam_MK5_MicroSD.sch (KiCad schematic (older format))
At the start: 3 parts, among them J8 DM3BT-DSF-PEJS, U9 MC74HC365ADG

Commit message: update
Parts:
- J8: symbol DM3BT-DSF-PEJS:DM3BT-DSF-PEJS -> SailCam_MK5-rescue:DM3BT-DSF-PEJS-DM3BT-DSF-PEJS
- U9: symbol MC74HC365ADG-ND:MC74HC365ADG -> SailCam_MK5-rescue:MC74HC365ADG-MC74HC365ADG-ND
Connections:
- net SD_MISO: now also U9.4 (A1); no longer U9.3 (Y0)
- net SD_MOSI: now also U9.3 (Y0); no longer U9.4 (A1)
Changed lines of the file:
@@
 $Descr A4 11693 8268
 encoding utf-8
-Sheet 7 7
+Sheet 6 7
 Title "SailCam"
 Date "2021-07-31"
@@
 $EndDescr
 $Comp
-L DM3BT-DSF-PEJS:DM3BT-DSF-PEJS J?
+L SailCam_MK5-rescue:DM3BT-DSF-PEJS-DM3BT-DSF-PEJS J?
 U 1 1 611DCAF8
 P 5050 2950
@@
 $EndComp
 $Comp
-L MC74HC365ADG-ND:MC74HC365ADG U?
+L SailCam_MK5-rescue:MC74HC365ADG-MC74HC365ADG-ND U?
 U 1 1 611DCAFF
 P 5150 4200
@@
 Text Label 5600 1650 0    50   ~ 0
 GND
+Text Label 5150 4500 2    50   ~ 0
+SD_MISO
 Text Label 5150 4400 2    50   ~ 0
-SD_MISO
-Text Label 5150 4500 2    50   ~ 0
 SD_MOSI
 Text Label 5150 4800 2    50   ~ 0

Commit message: hardward bug fixes
Parts:
- added R27: 10 KΩ, footprints:C_0805_2012Metric_Pad1.15x1.40mm_HandSolder_FullSilk, symbol Device:R_Small_US
Connections:
- net GND: now also J8.10 (CDSB); no longer U9.15 (OE2)
- net VCC: now also R27.1
- net at J8.9 (CDSA): now also U9.15 (OE2), R27.2
- no-connect marks 8 -> 6
Changed lines of the file:
@@
 Text Label 5150 4900 2    50   ~ 0
-GND
-Text Label 6750 4300 0    50   ~ 0
 GND
 Text Label 6850 3350 0    50   ~ 0
@@
 NoConn ~ 6850 3150
 NoConn ~ 5050 2950
-NoConn ~ 6850 3050
-NoConn ~ 6850 2950
 NoConn ~ 6750 4600
 NoConn ~ 6750 4700
@@
 	1    0    0    -1
 $EndComp
+$Comp
+L Device:R_Small_US R?
+U 1 1 624E72BB
+P 7000 4150
+AR Path="/624E72BB" Ref="R?"  Part="1"
+AR Path="/61217E38/624E72BB" Ref="R?"  Part="1"
+AR Path="/611DB121/624E72BB" Ref="R27"  Part="1"
+F 0 "R27" H 7068 4241 50  0000 L CNN
+F 1 "10 KΩ" H 7068 4150 50  0000 L CNN
+F 2 "footprints:C_0805_2012Metric_Pad1.15x1.40mm_HandSolder_FullSilk" H 7000 4150 50  0001 C CNN
+F 3 "~" H 7000 4150 50  0001 C CNN
+F 4 "5%" H 7068 4059 50  0000 L CNN "Tolerance"
+	1    7000 4150
+	1    0    0    -1
+$EndComp
+$Comp
+L power:VCC #PWR?
+U 1 1 624E72C1
+P 7000 4050
+AR Path="/624E72C1" Ref="#PWR?"  Part="1"
+AR Path="/611821E5/624E72C1" Ref="#PWR?"  Part="1"
+AR Path="/61199C7C/624E72C1" Ref="#PWR?"  Part="1"
+AR Path="/61217E38/624E72C1" Ref="#PWR?"  Part="1"
+AR Path="/611DB121/624E72C1" Ref="#PWR017"  Part="1"
+F 0 "#PWR017" H 7000 3900 50  0001 C CNN
+F 1 "VCC" H 7017 4223 50  0000 C CNN
+F 2 "" H 7000 4050 50  0001 C CNN
+F 3 "" H 7000 4050 50  0001 C CNN
+	1    7000 4050
+	1    0    0    -1
+$EndComp
+Wire Wire Line
+	6750 4300 7000 4300
+Wire Wire Line
+	7000 4300 7000 4250
+Wire Wire Line
+	7000 4300 7400 4300
+Wire Wire Line
+	7400 4300 7400 3050
+Wire Wire Line
+	7400 3050 6850 3050
+Connection ~ 7000 4300
+Text Label 6850 2950 0    50   ~ 0
+GND
 $EndSCHEMATC
