File: KiCad/SailCam_MK5/SailCam_MK5_PowerSupply.sch (KiCad schematic (older format))
At the start: 11 parts, among them U3 NCV7805BD2TG, U4 LTC4054ES5-4.2#TRMPBF, U5 XC6220B331MR-G

Commit message: update
Parts:
- U3: symbol NCV7805BD2TG:NCV7805BD2TG -> SailCam_MK5-rescue:NCV7805BD2TG-NCV7805BD2TG
- U4: symbol LTC4054ES5-4.2_TRMPBF:LTC4054ES5-4.2#TRMPBF -> SailCam_MK5-rescue:LTC4054ES5-4.2#TRMPBF-LTC4054ES5-4.2_TRMPBF
- U5: symbol XC6220B331MR-G:XC6220B331MR-G -> SailCam_MK5-rescue:XC6220B331MR-G-XC6220B331MR-G
Connections:
- net Bat_Chg_Vcc: now reaches C2.1, U3.3 (Output), U4.4 (VCC)
Changed lines of the file:
@@
 $EndDescr
 $Comp
-L XC6220B331MR-G:XC6220B331MR-G U?
+L SailCam_MK5-rescue:XC6220B331MR-G-XC6220B331MR-G U?
 U 1 1 611C1252
 P 6150 3100
@@
 Connection ~ 8050 3100
 $Comp
-L LTC4054ES5-4.2_TRMPBF:LTC4054ES5-4.2#TRMPBF U?
+L SailCam_MK5-rescue:LTC4054ES5-4.2#TRMPBF-LTC4054ES5-4.2_TRMPBF U?
 U 1 1 611C1280
 P 4600 4400
@@
 $EndComp
 $Comp
-L NCV7805BD2TG:NCV7805BD2TG U?
+L SailCam_MK5-rescue:NCV7805BD2TG-NCV7805BD2TG U?
 U 1 1 611C12B3
 P 3800 3100
@@
 Wire Wire Line
 	5750 3450 5750 2850
+Text HLabel 2000 1700 0    50   Input ~ 0
+Bat_Chg_Vcc
+Text Label 5600 4100 0    50   ~ 0
+Bat_Chg_Vcc
+Text Label 2000 1700 0    50   ~ 0
+Bat_Chg_Vcc
 $EndSCHEMATC

Commit message: mk5.2
Connections:
- net CHG: now also C1.1; no longer C1.2
- net GND: now also C1.2
- net VCC: no longer C1.1
Other:
- moved on the sheet: C1
Changed lines of the file:
@@
 L Device:C_Small C?
 U 1 1 611C12BC
-P 3800 2750
+P 3800 3200
 AR Path="/611C12BC" Ref="C?"  Part="1"
 AR Path="/611BA1F2/611C12BC" Ref="C1"  Part="1"
-F 0 "C1" H 3892 2796 50  0000 L CNN
-F 1 "0.33 uF" H 3892 2705 50  0000 L CNN
-F 2 "footprints:C_0805_2012Metric_Pad1.15x1.40mm_HandSolder_FullSilk" H 3800 2750 50  0001 C CNN
-F 3 "~" H 3800 2750 50  0001 C CNN
-	1    3800 2750
+F 0 "C1" H 3892 3246 50  0000 L CNN
+F 1 "0.33 uF" H 3892 3155 50  0000 L CNN
+F 2 "footprints:C_0805_2012Metric_Pad1.15x1.40mm_HandSolder_FullSilk" H 3800 3200 50  0001 C CNN
+F 3 "~" H 3800 3200 50  0001 C CNN
+	1    3800 3200
 	1    0    0    -1
 $EndComp
-$Comp
-L power:VCC #PWR?
-U 1 1 611C12C2
-P 3800 2650
-AR Path="/611C12C2" Ref="#PWR?"  Part="1"
-AR Path="/611BA1F2/611C12C2" Ref="#PWR0114"  Part="1"
-F 0 "#PWR0114" H 3800 2500 50  0001 C CNN
-F 1 "VCC" H 3817 2823 50  0000 C CNN
-F 2 "" H 3800 2650 50  0001 C CNN
-F 3 "" H 3800 2650 50  0001 C CNN
-	1    3800 2650
-	1    0    0    -1
-$EndComp
-Wire Wire Line
-	3800 2850 3800 3100
 Connection ~ 5600 4100
 Text Label 3800 3100 2    50   ~ 0
@@
 Text Label 2000 1700 0    50   ~ 0
 Bat_Chg_Vcc
+$Comp
+L power:GND #PWR?
+U 1 1 6153E2D4
+P 3800 3300
+F 0 "#PWR?" H 3800 3050 50  0001 C CNN
+F 1 "GND" H 3805 3127 50  0000 C CNN
+F 2 "" H 3800 3300 50  0001 C CNN
+F 3 "" H 3800 3300 50  0001 C CNN
+	1    3800 3300
+	1    0    0    -1
+$EndComp
 $EndSCHEMATC
